File: rp2040.brd (EAGLE design)
At the start: 55 x 25 mm, 58 parts, among them IC1 RP2040-QFN56, J2 1X6_2.5MM, J3 1X6_2.5MM, J4 1X6_2.5MM, J5 1X6_2.5MM, U1 9DoF IMU

Commit message: added bottom silk
Parts:
- moved U$3 0.08 mm to (55.0, 15.1)
Other:
- board text added: "0"
- board text added: "1"
- board text added: "1.1V"
- board text added: "10"
- board text added: "11"
- board text added: "12"
- board text added: "13"
- board text added: "14"
- board text added: "15"
- board text added: "16"
- board text added: "17"
- board text added: "18"
- board text added: "19"
- board text added: "2"
- board text added: "20"
- board text added: "21"
- board text added: "22"
- board text added: "23"
- board text added: "24"
- board text added: "25"
- board text added: "26/ADC0"
- board text added: "27/ADC1"
- board text added: "28/ADC2"
- board text added: "29/ADC3"
- board text added: "3"
- board text added: "3.3V"
- board text added: "4"
- board text added: "5/IMU_INT"
- board text added: "5V"
- board text added: "6/SDA1"
- board text added: "7/SCL1"
- board text added: "8"
- board text added: "9"
- board text added: "BOOT"
- board text added: "GND"
- board text added: "RUN"
- board text added: "SWCLK"
- board text added: "SWD"
